File: kicad/NanoUPDI_v2.kicad_sch (KiCad schematic)
At the start: 20 parts, among them J1 Conn_01x03, SW1 VCC, U1 CH340E

Commit message: Update Kicad Schematic
Parts:
- C1: value 100nF -> 100n
- SW1: value VCC -> MSK12C02
Other:
- moved on the sheet: SW1
Changed lines of the file:
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@@
 	(wire
 		(pts
-			(xy 217.17 139.7) (xy 217.17 140.335)
+			(xy 217.17 140.97) (xy 217.17 141.605)
 		)
 		(stroke
@@
 	(wire
 		(pts
-			(xy 217.17 145.415) (xy 215.265 145.415)
+			(xy 217.17 146.685) (xy 215.265 146.685)
 		)
 		(stroke
@@
 	(wire
 		(pts
-			(xy 204.47 142.24) (xy 204.47 142.875)
-		)
-		(stroke
-			(width 0)
-			(type default)
-		)
-	)
-	(wire
-		(pts
-			(xy 217.17 140.335) (xy 215.265 140.335)
+			(xy 204.47 143.51) (xy 204.47 144.145)
+		)
+		(stroke
+			(width 0)
+			(type default)
+		)
+	)
+	(wire
+		(pts
+			(xy 217.17 141.605) (xy 215.265 141.605)
 		)
 		(stroke
@@
 	(wire
 		(pts
-			(xy 204.47 142.875) (xy 205.105 142.875)
+			(xy 204.47 144.145) (xy 205.105 144.145)
 		)
 		(stroke
@@
 	(symbol
 		(lib_id "power:+3V3")
-		(at 217.17 139.7 0)
+		(at 217.17 140.97 0)
 		(unit 1)
 		(exclude_from_sim no)
@@
 		(fields_autoplaced yes)
 		(property "Reference" "#PWR013"
-			(at 217.17 143.51 0)
+			(at 217.17 144.78 0)
 			(effects
 				(font
@@
 		)
 		(property "Value" "+3V3"
-			(at 217.17 136.525 0)
+			(at 217.17 137.795 0)
 			(effects
 				(font
@@
 		)
 		(property "Footprint" ""
-			(at 217.17 139.7 0)
+			(at 217.17 140.97 0)
 			(effects
 				(font
@@
 		)
 		(property "Datasheet" ""
-			(at 217.17 139.7 0)
+			(at 217.17 140.97 0)
 			(effects
 				(font
@@
 		)
 		(property "Description" ""
-			(at 217.17 139.7 0)
+			(at 217.17 140.97 0)
 			(effects
 				(font
@@
 	(symbol
 		(lib_id "Switch:SW_SPDT")
-		(at 210.185 142.875 0)
+		(at 210.185 144.145 0)
 		(unit 1)
 		(exclude_from_sim no)
@@
 		(dnp no)
 		(property "Reference" "SW1"
-			(at 210.185 136.525 0)
-			(effects
-				(font
-					(size 1.27 1.27)
-				)
-			)
-		)
-		(property "Value" "VCC"
-			(at 210.185 138.43 0)
+			(at 210.185 133.985 0)
+			(effects
+				(font
+					(size 1.27 1.27)
+				)
+			)
+		)
+		(property "Value" "MSK12C02"
+			(at 210.185 135.89 0)
 			(effects
 				(font
@@
 		)
 		(property "Footprint" "MSK12C02:MSK12C02"
-			(at 210.185 142.875 0)
+			(at 210.185 144.145 0)
 			(effects
 				(font
@@
 		)
 		(property "Datasheet" "~"
-			(at 210.185 142.875 0)
+			(at 210.185 144.145 0)
 			(effects
 				(font
@@
 		)
 		(property "Description" ""
-			(at 210.185 142.875 0)
+			(at 210.185 144.145 0)
 			(effects
 				(font
@@
 	(symbol
 		(lib_id "power:+5V")
-		(at 217.17 145.415 0)
+		(at 217.17 146.685 0)
 		(unit 1)
 		(exclude_from_sim no)
@@
 		(dnp no)
 		(property "Reference" "#PWR02"
-			(at 217.17 149.225 0)
+			(at 217.17 150.495 0)
 			(effects
 				(font
@@
 		)
 		(property "Value" "+5V"
-			(at 217.17 141.605 0)
+			(at 217.17 142.875 0)
 			(effects
 				(font
@@
 		)
 		(property "Footprint" ""
-			(at 217.17 145.415 0)
+			(at 217.17 146.685 0)
 			(effects
 				(font
@@
 		)
 		(property "Datasheet" ""
-			(at 217.17 145.415 0)
+			(at 217.17 146.685 0)
 			(effects
 				(font
@@
 		)
 		(property "Description" ""
-			(at 217.17 145.415 0)
+			(at 217.17 146.685 0)
 			(effects
 				(font
@@
 		(fields_autoplaced yes)
 		(property "Reference" "C1"
-			(at 98.425 44.4563 0)
+			(at 97.79 43.8212 0)
 			(effects
 				(font
@@
 			)
 		)
-		(property "Value" "100nF"
-			(at 98.425 46.9963 0)
+		(property "Value" "100n"
+			(at 97.79 46.3612 0)
 			(effects
 				(font
@@
 	(symbol
 		(lib_id "power:VCC")
-		(at 204.47 142.24 0)
+		(at 204.47 143.51 0)
 		(unit 1)
 		(exclude_from_sim no)
@@
 		(dnp no)
 		(property "Reference" "#PWR022"
-			(at 204.47 146.05 0)
+			(at 204.47 147.32 0)
 			(effects
 				(font
@@
 		)
 		(property "Value" "VCC"
-			(at 204.47 138.43 0)
+			(at 204.47 139.7 0)
 			(effects
 				(font
@@
 		)
 		(property "Footprint" ""
-			(at 204.47 142.24 0)
+			(at 204.47 143.51 0)
 			(effects
 				(font
@@
 		)
 		(property "Datasheet" ""
-			(at 204.47 142.24 0)
+			(at 204.47 143.51 0)
 			(effects
 				(font
@@
 		)
 		(property "Description" ""
-			(at 204.47 142.24 0)
-			(effects
-				(font
+			(at 204.47 143.51 0)
+			(effects
+				(font
